File: hardware/laemp_pcb/laemp/power.kicad_sch (KiCad schematic)
At the start: 43 parts, among them U2 TPS61165DRV, U3 TPS61165DRV, U4 TPS61165DRV, U6 TPS61165DRV

Commit message: updated schematic
Parts:
- added C18, C19, C20, C21: 220nF, Capacitor_SMD:C_0603_1608Metric, symbol Device:C
- added C22: 220uF 25V, symbol Device:C_Polarized
- C10, C12, C6, C8: value C -> 10uF 50V X7R
- C11, C5, C7, C9: value C -> 4.7uF 50V X7R; footprint (none) -> Capacitor_SMD:C_0805_2012Metric
- D1, D13, D17, D9: value D_Schottky -> SOD123F
- L2, L3, L4, L5: value L -> 22uH
- R3: value R -> 0.56R; footprint (none) -> Resistor_SMD:R_1206_3216Metric
- R4, R5, R6: value R -> 0.62R; footprint (none) -> Resistor_SMD:R_1206_3216Metric
Connections:
- net +15V: now also C22.1
- net AGND: now also C10.2, C11.2, C5.2, C7.2, C9.2, R3.2, R4.2, R5.2, R6.2, U2.3 (GND), U2.7 (GND), U3.3 (GND), U3.7 (GND), U4.3 (GND), U4.7 (GND), U6.3 (GND), U6.7 (GND), C18.2, C19.2, C20.2, C21.2, C22.2
- net GND: no longer C10.2, C11.2, C5.2, C7.2, C9.2, R3.2, R4.2, R5.2, R6.2, U2.3 (GND), U2.7 (GND), U3.3 (GND), U3.7 (GND), U4.3 (GND), U4.7 (GND), U6.3 (GND), U6.7 (GND)
- net at U4.2 (COMP): now also C19.1
- net at U6.2 (COMP): now also C18.1
- net at U3.2 (COMP): now also C21.1
- net at U2.2 (COMP): now also C20.1
Other:
- moved on the sheet: C11, C5, C7, C9, R3, R4, R5, R6

Commit message: added more footprints
Parts:
- C13, C17: footprint (none) -> Capacitor_SMD:C_0603_1608Metric
- R10, R7, R8, R9: footprint (none) -> Resistor_SMD:R_0603_1608Metric
Changed lines of the file:
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@@
 			)
 		)
-		(property "Footprint" ""
+		(property "Footprint" "Resistor_SMD:R_0603_1608Metric"
 			(at 308.61 94.488 90)
 			(hide yes)
@@
 			)
 		)
-		(property "Footprint" ""
+		(property "Footprint" "Capacitor_SMD:C_0603_1608Metric"
 			(at 319.7352 55.88 0)
 			(hide yes)
@@
 			)
 		)
-		(property "Footprint" ""
+		(property "Footprint" "Capacitor_SMD:C_0603_1608Metric"
 			(at 257.5052 77.47 0)
 			(hide yes)
@@
 			)
 		)
-		(property "Footprint" ""
+		(property "Footprint" "Resistor_SMD:R_0603_1608Metric"
 			(at 271.272 86.36 90)
 			(hide yes)
@@
 			)
 		)
-		(property "Footprint" ""
+		(property "Footprint" "Resistor_SMD:R_0603_1608Metric"
 			(at 348.742 74.93 90)
 			(hide yes)
@@
 			)
 		)
-		(property "Footprint" ""
+		(property "Footprint" "Resistor_SMD:R_0603_1608Metric"
 			(at 348.742 86.36 90)
 			(hide yes)

Commit message: added inductor footprint
Parts:
- L2, L3, L4, L5: footprint (none) -> Inductor_SMD:L_Vishay_IHLP-4040
Changed lines of the file:
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@@
 	(text "NEEDS THERMAL VIAS"
 		(exclude_from_sim no)
-		(at 65.786 25.908 0)
+		(at 71.12 24.13 0)
 		(effects
 			(font
@@
 			)
 		)
-		(property "Footprint" ""
+		(property "Footprint" "Inductor_SMD:L_Vishay_IHLP-4040"
 			(at 163.83 31.75 0)
 			(hide yes)
@@
 			)
 		)
-		(property "Footprint" ""
+		(property "Footprint" "Inductor_SMD:L_Vishay_IHLP-4040"
 			(at 67.31 99.06 0)
 			(hide yes)
@@
 			)
 		)
-		(property "Footprint" ""
+		(property "Footprint" "Inductor_SMD:L_Vishay_IHLP-4040"
 			(at 68.58 33.02 0)
 			(hide yes)
@@
 			)
 		)
-		(property "Footprint" ""
+		(property "Footprint" "Inductor_SMD:L_Vishay_IHLP-4040"
 			(at 162.56 101.6 0)
 			(hide yes)
